File: XY_Faces/solar-panel-NoCutout.kicad_pcb (KiCad board)
At the start: 4 copper layers, 83 x 98 mm, 25 parts, among them J1 CON-5040500591, J2 Conn_01x01, J3 Conn_01x01, J4 Conn_01x01, J5 Conn_01x01, U1 VEML7700, U2 MCP9808_DFN, U3 DRV2605LDGS

Commit message: removed coil wires, may have power conenctions that need to be removed and etc
Routing:
- net Net-(U3-Pad7): track 8719.1 -> 75.4 mm
